File: kicad_file/Buzzer_JHE42B.sch (KiCad schematic (older format))
At the start: 18 parts, among them SW1 SW_Push

Commit message: update and rename of schematic files
Parts:
- Remote: renamed from RemoteHeader; value Buzz/5V/GND -> Header
- gave numbers to parts that had none: 1
Other:
- moved on the sheet: 1AM, 2.2Ohm, 9.45kOhm, 980Ohm, BuzzerLight, Diode1, PowerOn, R1, R2, Remote, SW1
Changed lines of the file:
@@
 encoding utf-8
 Sheet 1 1
-Title ""
-Date ""
-Rev ""
-Comp ""
-Comment1 ""
+Title "Autonomous Buzzer JHE42B"
+Date "2021-02-0"
+Rev "3"
+Comp "Reversed schematic"
+Comment1 "Needs to be double checked"
 Comment2 ""
 Comment3 ""
@@
 	5150 4000 5550 4000
 Wire Wire Line
-	5550 3000 6150 3000
+	4800 3000 6150 3000
 $Comp
 L Device:R_Small R2
 U 1 1 601A0ACE
-P 5450 3000
-F 0 "R2" V 5646 3000 50  0000 C CNN
-F 1 "9.94Kohm" V 5555 3000 50  0000 C CNN
-F 2 "" H 5450 3000 50  0001 C CNN
-F 3 "~" H 5450 3000 50  0001 C CNN
-	1    5450 3000
+P 4700 3000
+F 0 "R2" V 4896 3000 50  0000 C CNN
+F 1 "9.94Kohm" V 4805 3000 50  0000 C CNN
+F 2 "" H 4700 3000 50  0001 C CNN
+F 3 "~" H 4700 3000 50  0001 C CNN
+	1    4700 3000
 	0    1    -1   0
 $EndComp
@@
 L Device:LED BuzzerLight
 U 1 1 6014D1A4
-P 3850 4750
-F 0 "BuzzerLight" H 3843 4967 50  0000 C CNN
-F 1 "LED" H 3843 4876 50  0000 C CNN
-F 2 "" H 3850 4750 50  0001 C CNN
-F 3 "~" H 3850 4750 50  0001 C CNN
-	1    3850 4750
+P 3850 4400
+F 0 "BuzzerLight" H 3843 4617 50  0000 C CNN
+F 1 "LED" H 3843 4526 50  0000 C CNN
+F 2 "" H 3850 4400 50  0001 C CNN
+F 3 "~" H 3850 4400 50  0001 C CNN
+	1    3850 4400
 	-1   0    0    1
 $EndComp
@@
 L Device:R_Small 2.2Ohm
 U 1 1 60150121
-P 3600 4750
-F 0 "2.2Ohm" V 3700 4750 50  0000 C CNN
-F 1 "R_shunt 62R0" V 3800 4750 50  0000 C CNN
-F 2 "" H 3600 4750 50  0001 C CNN
-F 3 "~" H 3600 4750 50  0001 C CNN
-	1    3600 4750
+P 3600 4400
+F 0 "2.2Ohm" V 3700 4400 50  0000 C CNN
+F 1 "R_shunt 62R0" V 3800 4400 50  0000 C CNN
+F 2 "" H 3600 4400 50  0001 C CNN
+F 3 "~" H 3600 4400 50  0001 C CNN
+	1    3600 4400
 	0    1    -1   0
 $EndComp
@@
 L Diode:1N5819 Diode1
 U 1 1 60158A46
-P 3350 4750
-F 0 "Diode1" H 3350 4900 50  0000 C CNN
-F 1 "||SL - 1N5819" H 3450 5000 50  0000 C CNN
-F 2 "Diode_THT:D_DO-41_SOD81_P10.16mm_Horizontal" H 3350 4575 50  0001 C CNN
-F 3 "http://www.vishay.com/docs/88525/1n5817.pdf" H 3350 4750 50  0001 C CNN
-	1    3350 4750
+P 3350 4400
+F 0 "Diode1" H 3350 4550 50  0000 C CNN
+F 1 "||SL - 1N5819" H 3450 4650 50  0000 C CNN
+F 2 "Diode_THT:D_DO-41_SOD81_P10.16mm_Horizontal" H 3350 4225 50  0001 C CNN
+F 3 "http://www.vishay.com/docs/88525/1n5817.pdf" H 3350 4400 50  0001 C CNN
+	1    3350 4400
 	-1   0    0    1
 $EndComp
@@
 	1    0    0    -1
 $EndComp
-Wire Wire Line
-	5550 3400 4750 3400
 $Comp
 L Device:R_Small 2.2Ohm
@@
 L Transistor_BJT:MMBT3904 1AM
 U 1 1 601218E6
-P 4200 4750
-F 0 "1AM" V 4435 4750 50  0000 C CNN
-F 1 "MMBT3904" V 4526 4750 50  0000 C CNN
-F 2 "Package_TO_SOT_SMD:SOT-23" H 4400 4675 50  0001 L CIN
-F 3 "https://www.onsemi.com/pub/Collateral/2N3903-D.PDF" H 4200 4750 50  0001 L CNN
-	1    4200 4750
+P 4200 4400
+F 0 "1AM" H 4550 4350 50  0000 C CNN
+F 1 "MMBT3904" H 4600 4500 50  0000 C CNN
+F 2 "Package_TO_SOT_SMD:SOT-23" H 4400 4325 50  0001 L CIN
+F 3 "https://www.onsemi.com/pub/Collateral/2N3903-D.PDF" H 4200 4400 50  0001 L CNN
+	1    4200 4400
 	1    0    0    1
 $EndComp
@@
 L power:GND #PWR?
 U 1 1 601E26E8
-P 4300 4950
-F 0 "#PWR?" H 4300 4700 50  0001 C CNN
-F 1 "GND" H 4305 4777 50  0000 C CNN
-F 2 "" H 4300 4950 50  0001 C CNN
-F 3 "" H 4300 4950 50  0001 C CNN
-	1    4300 4950
+P 4300 4600
+F 0 "#PWR?" H 4300 4350 50  0001 C CNN
+F 1 "GND" H 4305 4427 50  0000 C CNN
+F 2 "" H 4300 4600 50  0001 C CNN
+F 3 "" H 4300 4600 50  0001 C CNN
+	1    4300 4600
 	1    0    0    -1
 $EndComp
@@
 L Device:R_Small R1
 U 1 1 6017D0ED
-P 7750 4600
-F 0 "R1" V 7946 4600 50  0000 C CNN
-F 1 "9.94Kohm" V 7855 4600 50  0000 C CNN
-F 2 "" H 7750 4600 50  0001 C CNN
-F 3 "~" H 7750 4600 50  0001 C CNN
-	1    7750 4600
+P 7650 4600
+F 0 "R1" V 7846 4600 50  0000 C CNN
+F 1 "9.94Kohm" V 7755 4600 50  0000 C CNN
+F 2 "" H 7650 4600 50  0001 C CNN
+F 3 "~" H 7650 4600 50  0001 C CNN
+	1    7650 4600
 	0    1    -1   0
 $EndComp
@@
 	6750 4000 7400 4000
 Wire Wire Line
-	7650 4600 7400 4600
+	7550 4600 7400 4600
 Wire Wire Line
 	7400 4600 7400 4000
@@
 	7400 4000 7500 4000
 Wire Wire Line
-	7850 4600 7900 4600
+	7750 4600 7900 4600
 Wire Wire Line
 	7900 4600 7900 4000
 Connection ~ 7900 4600
 $Comp
-L Transistor_FET:BSN20 Q?
+L Transistor_FET:BSN20 Q
 U 1 1 6018635A
 P 7700 3900
-F 0 "Q?" H 7905 3946 50  0000 L CNN
-F 1 "BSN20" H 7905 3855 50  0000 L CNN
+F 0 "Q" V 7700 3650 50  0000 L CNN
+F 1 "BSN20" V 7600 3600 50  0000 L CNN
 F 2 "Package_TO_SOT_SMD:SOT-23" H 7900 3825 50  0001 L CIN
 F 3 "http://www.diodes.com/assets/Datasheets/ds31898.pdf" H 7700 3900 50  0001 L CNN
@@
 	7700 3300 7700 3500
 Wire Wire Line
-	5350 3000 2300 3000
+	4600 3000 2250 3000
 $Comp
 L power:GND #PWR?
 U 1 1 602456CD
-P 2300 3200
-F 0 "#PWR?" H 2300 2950 50  0001 C CNN
-F 1 "GND" H 2300 3000 50  0000 C CNN
-F 2 "" H 2300 3200 50  0001 C CNN
-F 3 "" H 2300 3200 50  0001 C CNN
-	1    2300 3200
+P 2250 3200
+F 0 "#PWR?" H 2250 2950 50  0001 C CNN
+F 1 "GND" H 2250 3000 50  0000 C CNN
+F 2 "" H 2250 3200 50  0001 C CNN
+F 3 "" H 2250 3200 50  0001 C CNN
+	1    2250 3200
 	1    0    0    -1
 $EndComp
@@
 L Device:LED PowerOn
 U 1 1 6024A005
-P 2650 3100
-F 0 "PowerOn" H 2700 3350 50  0000 C CNN
-F 1 "LED" H 2700 3250 50  0000 C CNN
-F 2 "" H 2650 3100 50  0001 C CNN
-F 3 "~" H 2650 3100 50  0001 C CNN
-	1    2650 3100
+P 2650 3400
+F 0 "PowerOn" H 2700 3650 50  0000 C CNN
+F 1 "LED" H 2700 3550 50  0000 C CNN
+F 2 "" H 2650 3400 50  0001 C CNN
+F 3 "~" H 2650 3400 50  0001 C CNN
+	1    2650 3400
 	-1   0    0    1
 $EndComp
@@
 L Device:R_Small 980Ohm
 U 1 1 6024A00B
-P 2900 3100
-F 0 "980Ohm" V 2700 3150 50  0000 C CNN
-F 1 "R5" V 2800 3100 50  0000 C CNN
-F 2 "" H 2900 3100 50  0001 C CNN
-F 3 "~" H 2900 3100 50  0001 C CNN
-	1    2900 3100
-	0    1    -1   0
-$EndComp
-Wire Wire Line
-	2300 3100 2500 3100
-$Comp
-L Connector_Generic:Conn_01x03 RemoteHeader
+P 2900 3400
+F 0 "980Ohm" V 2700 3450 50  0000 C CNN
+F 1 "R5" V 2800 3400 50  0000 C CNN
+F 2 "" H 2900 3400 50  0001 C CNN
+F 3 "~" H 2900 3400 50  0001 C CNN
+	1    2900 3400
+	0    1    -1   0
+$EndComp
+$Comp
+L Connector_Generic:Conn_01x03 Remote
 U 1 1 6023EF45
-P 2100 3100
-F 0 "RemoteHeader" H 2600 3350 50  0000 R CNN
-F 1 "Buzz/5V/GND" H 2700 3000 50  0000 R CNN
-F 2 "" H 2100 3100 50  0001 C CNN
-F 3 "~" H 2100 3100 50  0001 C CNN
-	1    2100 3100
+P 2050 3100
+F 0 "Remote" H 2450 3450 50  0000 R CNN
+F 1 "Header" H 2450 3350 50  0000 R CNN
+F 2 "" H 2050 3100 50  0001 C CNN
+F 3 "~" H 2050 3100 50  0001 C CNN
+	1    2050 3100
 	-1   0    0    -1
 $EndComp
@@
 L power:GND #PWR?
 U 1 1 601CA5AE
-P 3750 3750
-F 0 "#PWR?" H 3750 3500 50  0001 C CNN
-F 1 "GND" H 3755 3577 50  0000 C CNN
-F 2 "" H 3750 3750 50  0001 C CNN
-F 3 "" H 3750 3750 50  0001 C CNN
-	1    3750 3750
+P 4100 3750
+F 0 "#PWR?" H 4100 3500 50  0001 C CNN
+F 1 "GND" H 4105 3577 50  0000 C CNN
+F 2 "" H 4100 3750 50  0001 C CNN
+F 3 "" H 4100 3750 50  0001 C CNN
+	1    4100 3750
 	1    0    0    -1
 $EndComp
@@
 L Switch:SW_Push SW1
 U 1 1 6013F9ED
-P 3950 3750
-F 0 "SW1" H 3950 4035 50  0000 C CNN
-F 1 "SW_Push" H 3950 3944 50  0000 C CNN
-F 2 "" H 3950 3950 50  0001 C CNN
-F 3 "~" H 3950 3950 50  0001 C CNN
-	1    3950 3750
+P 4300 3750
+F 0 "SW1" H 4300 4035 50  0000 C CNN
+F 1 "SW_Push" H 4300 3944 50  0000 C CNN
+F 2 "" H 4300 3950 50  0001 C CNN
+F 3 "~" H 4300 3950 50  0001 C CNN
+	1    4300 3750
 	1    0    0    -1
 $EndComp
@@
 L Device:R_Small 9.45kOhm
 U 1 1 601376D3
-P 3550 3100
-F 0 "9.45kOhm" V 3350 3100 50  0000 C CNN
-F 1 "R4" V 3450 3100 50  0000 C CNN
-F 2 "" H 3550 3100 50  0001 C CNN
-F 3 "~" H 3550 3100 50  0001 C CNN
-	1    3550 3100
-	0    1    -1   0
-$EndComp
-Wire Wire Line
-	4750 3100 4750 3400
-Wire Wire Line
-	3650 3100 4750 3100
-Wire Wire Line
-	4150 3750 4950 3750
+P 3650 3400
+F 0 "9.45kOhm" V 3450 3400 50  0000 C CNN
+F 1 "R4" V 3550 3400 50  0000 C CNN
+F 2 "" H 3650 3400 50  0001 C CNN
+F 3 "~" H 3650 3400 50  0001 C CNN
+	1    3650 3400
+	0    1    -1   0
+$EndComp
+Wire Wire Line
+	4500 3750 4950 3750
 Wire Wire Line
 	4950 3750 4950 3500
@@
 	4950 3500 5550 3500
 Wire Wire Line
-	3000 3100 3200 3100
-Wire Wire Line
-	3200 4750 3200 3100
-Connection ~ 3200 3100
-Wire Wire Line
-	3200 3100 3450 3100
-Wire Wire Line
-	4300 4550 4300 4000
+	3000 3400 3200 3400
+Wire Wire Line
+	3200 4400 3200 3400
+Connection ~ 3200 3400
+Wire Wire Line
+	3200 3400 3550 3400
+Wire Wire Line
+	4300 4200 4300 4000
 Wire Wire Line
 	4300 4000 4950 4000
+Text Label 1700 3050 0    50   ~ 0
+Buzzer
+Text Label 1850 3150 0    50   ~ 0
+5V
+Text Label 1800 3250 0    50   ~ 0
+GND
+Wire Wire Line
+	3750 3400 5550 3400
+Wire Wire Line
+	2250 3100 2500 3100
+Wire Wire Line
+	2500 3100 2500 3400
 $EndSCHEMATC

Commit message: schematic changes
Changed lines of the file:
@@
 Sheet 1 1
 Title "Autonomous Buzzer JHE42B"
-Date "2021-02-0"
-Rev "3"
+Date "2021-02-05"
+Rev "4"
 Comp "Reversed schematic"
 Comment1 "Needs to be double checked"
@@
 P 8850 4550
 F 0 "VoltReg_662k" H 8850 4792 50  0000 C CNN
-F 1 "XC6206PxxxMR 5vTo3.3v" H 8850 4701 50  0000 C CNN
+F 1 "XC6206PxxxMR 5vTo3.3v" H 8850 4700 50  0000 C CNN
 F 2 "Package_TO_SOT_SMD:SOT-23" H 8850 4775 50  0001 C CIN
 F 3 "https://www.torexsemi.com/file/xc6206/XC6206.pdf" H 8850 4550 50  0001 C CNN
